Commit message: Rope added (4 links, and 3 joints) + sphere that represents load. Which joint to use? Reference for physics? How to offset links and joints?

File: morus_description/urdf/morus.base.urdf.xacro (robot description, xacro)
@@ -16,5 +16,5 @@
   <xacro:property name="motor_constant" value="0.000456874" /> <!-- [kg*m/s^2] -->
   <xacro:property name="moment_constant" value="0.01" /> <!-- [m] -->
-  <xacro:property name="time_constant" value="0.125" /> <!-- [s] -->s ti
+  <xacro:property name="time_constant" value="0.125" /> <!-- [s] -->
   <xacro:property name="max_rot_velocity" value="838" /> <!-- [rad/s] -->
   <xacro:property name="rotor_drag_coefficient" value="8.06428e-04" />
