Commit message: Mesh visuals commented for easier moddeling

File: morus_description/urdf/multirotor_base.urdf.xacro (robot description, xacro)
@@ -16,12 +16,12 @@
         <xacro:insert_block name="inertia" />
       </inertial>
-      <visual>
+      <!--visual>
         <origin xyz="0 0 0.125" rpy="0 0 0" />
         <geometry>
           <mesh filename="package://morus_description/meshes/${mesh_file}"
             scale="1 1 1" />
-          <!--box size="${body_width} ${body_width} ${body_height}"/--> <!-- [m] [m] [m] -->
-        </geometry>
-      </visual>
+          <box size="${body_width} ${body_width} ${body_height}"/--> <!-- [m] [m] [m] -->
+        <!--/geometry>
+      </visual-->
       <collision>
         <origin xyz="0 0 0" rpy="0 0 0" />

Commit message: Removing mesh for easier modelling

File: morus_description/urdf/multirotor_base.urdf.xacro (robot description, xacro)
@@ -16,12 +16,12 @@
         <xacro:insert_block name="inertia" />
       </inertial>
-      <!--visual>
+      <visual>
         <origin xyz="0 0 0.125" rpy="0 0 0" />
         <geometry>
-          <mesh filename="package://morus_description/meshes/${mesh_file}"
-            scale="1 1 1" />
-          <box size="${body_width} ${body_width} ${body_height}"/--> <!-- [m] [m] [m] -->
-        <!--/geometry>
-      </visual-->
+          <!--mesh filename="package://morus_description/meshes/${mesh_file}"
+            scale="1 1 1" /-->
+          <!--box size="${body_width} ${body_width} ${body_height}"/--> <!-- [m] [m] [m] -->
+        </geometry>
+      </visual>
       <collision>
         <origin xyz="0 0 0" rpy="0 0 0" />

Commit message: Modified code (added rope and load) Which joints to use? How to represent rope (physical aspect)? Physical attributes of drone. Offset of transfer frames?

File: morus_description/urdf/multirotor_base.urdf.xacro (robot description, xacro)
@@ -4,4 +4,13 @@
   <xacro:macro name="multirotor_base_macro"
     params="robot_namespace mass body_width body_height mesh_file mesh_file_mass *inertia">
+		<material name="blue">
+   	  <color rgba="0 0 0.8 1"/>
+    </material>
+   	<material name="green">
+   		<color rgba="0 0.8 0 1"/>
+		</material>
+		<material name="red">
+   		<color rgba="0.8 0 0 1"/>
+		</material>
     <link name="base_link"></link>
     <joint name="base_joint" type="fixed">
@@ -19,6 +28,6 @@
         <origin xyz="0 0 0.125" rpy="0 0 0" />
         <geometry>
-          <!--mesh filename="package://morus_description/meshes/${mesh_file}"
-            scale="1 1 1" /-->
+          <mesh filename="package://morus_description/meshes/${mesh_file}"
+            scale="1 1 1" />		<!-- zakomentirati ovaj mesh za jednostavniju izvedbu  -->
           <!--box size="${body_width} ${body_width} ${body_height}"/--> <!-- [m] [m] [m] -->
         </geometry>
@@ -45,6 +54,137 @@
       <parent link="base_link" />
       <child link="imu_link" />
-      <limit upper="0" lower="0" effort="0" velocity="0" />
-    </joint>
+      <limit upper="0" lower="0" effort="0" velocity="0" />  		<!-- kako funkcioniraju ova  ogranicenja?-->
+		</joint>
+		<!-- Rope addition-->
+		<link name="rope_1">
+			<collision>
+				<geometry>
+					<cylinder length="0.1" radius="0.01"/>
+				</geometry>
+				<material name="red"/>
+			</collision>
+			<visual>
+				<geometry>
+					<cylinder length="0.1" radius="0.01"/>
+				</geometry>
+				<material name="red"/>
+			</visual>
+			<inertial>
+				<mass value="0.01"/>
+				<inertia
+					ixx="0.01" ixy="0.0" ixz="0.0"
+        	iyy="0.01" iyz="0.0"
+        	izz="0.01"/>
+				</inertial>
+		</link>
+		<joint name="base_to_rope" type="fixed">
+			<parent link="base_link"/>
+			<child link="rope_1"/>
+			<origin xyz="0 0 -0.15" rpy="0 0 0"/>  <!--kako se gleda offset kod jointova, odnosno koji je reference tf-->
+		</joint>
+	<link name="rope_2">
+			<collision>
+				<geometry>
+					<box size="0.01 0.01 0.1"/>
+				</geometry>
+			</collision>
+			<visual>
+				<geometry>
+					<box size="0.01 0.01 0.1"/>
+				</geometry>
+				<material name="blue"/>
+			</visual>
+			<inertial>
+				<mass value="0.01"/>
+				<inertia
+					ixx="0.01" ixy="0.0" ixz="0.0"
+        	iyy="0.01" iyz="0.0"
+        	izz="0.01"/>
+				</inertial>
+		</link>
+		<joint name="rope1_to_rope2" type="revolute">
+			<parent link="rope_1"/>
+			<child link="rope_2"/>
+			<origin xyz="0 0 -0.1" rpy="0 0 0"/>
+			<limit upper="1" lower="1" effort="5" velocity="5" />
+			<axis xyz="1 1 0"/>
+		</joint>
+	<link name="rope_3">
+			<collision>
+				<geometry>
+					<box size="0.005 0.005 0.1"/>
+				</geometry>
+			</collision>
+			<visual>
+				<geometry>
+					<box size="0.005 0.005 0.1"/>
+				</geometry>
+				<material name="green"/>
+			</visual>
+			<inertial>
+				<mass value="0.01"/>
+				<inertia
+					ixx="0.01" ixy="0.0" ixz="0.0"
+        	iyy="0.01" iyz="0.0"
+        	izz="0.01"/>
+				</inertial>
+		</link>
+		<joint name="rope2_to_rope3" type="revolute">
+			<parent link="rope_2"/>
+			<child link="rope_3"/>
+			<origin xyz="0 0 -0.1" rpy="0 0 0"/>
+			<limit upper="1.5707" lower="1.5707" effort="5" velocity="5" />
+			<axis xyz="1 1 0"/>
+		</joint>
+			<link name="rope_4">
+			<collision>
+				<geometry>
+					<cylinder radius ="0.0025" length="0.15"/>
+				</geometry>
+			</collision>
+			<visual>
+				<geometry>
+					<cylinder radius ="0.0025" length="0.15"/>
+				</geometry>
+			</visual>
+			<inertial>
+				<mass value="0.01"/>
+				<inertia
+					ixx="0.01" ixy="0.0" ixz="0.0"
+        	iyy="0.01" iyz="0.0"
+        	izz="0.01"/>
+				</inertial>
+		</link>
+		<joint name="rope3_to_rope4" type="revolute">			<!-- na koji nacin modelirati zglobove -->
+			<parent link="rope_3"/>
+			<child link="rope_4"/>
+			<origin xyz="0 0 -0.1" rpy="0 0 0"/>
+			<limit upper="1.5707" lower="1.5707" effort="5" velocity="5" />   	<!-- kako im postaviti ogranicenja -->
+			<axis xyz="1 1 0"/>
+		</joint>
+		<link name="load">
+			<collision>
+				<geometry>
+					<sphere radius ="0.075" />
+				</geometry>
+			</collision>
+			<visual>
+				<geometry>
+					<sphere radius ="0.075" />
+				</geometry>
+			</visual>
+			<inertial>
+				<mass value="0.25"/>
+				<inertia
+					ixx="0.05" ixy="0.0" ixz="0.0"
+        	iyy="0.05" iyz="0.0"
+        	izz="0.05"/>
+				</inertial>
+		</link>
+		<joint name="rope4_to_load" type="fixed">
+			<parent link="rope_4"/>
+			<child link="load"/>
+			<origin xyz="0 0 -0.15" rpy="0 0 0"/>
+		</joint>
     <!-- attach multirotor_base_plugin to the base_link -->
     <gazebo>
@@ -75,5 +215,5 @@
           <!--mesh filename="package://morus_description/meshes/${mesh_file_mass}"
             scale="1 1 1" /-->
-          <box size="${1*dimension} ${1*dimension} ${1*dimension}"/>
+          <!--box size="${1*dimension} ${1*dimension} ${1*dimension}"/-->
         </geometry>
       </visual>
@@ -81,5 +221,5 @@
         <origin rpy="0 0 0" xyz="0 0 ${0*movable_mass_dimension/2}"/>
         <geometry>
-          <box size="${dimension} ${dimension} ${dimension}"/>
+          <!--box size="${dimension} ${dimension} ${dimension}"/-->
         </geometry>
       </collision>
@@ -115,7 +255,7 @@
       <visual>
         <geometry>
-          <!-- <cylinder length="0.005" radius="${radius_rotor}"/> --> <!-- [m] -->
-          <mesh filename="package://morus_description/meshes/propeller_${direction}.dae"
-            scale="0.0025 0.0025 0.0025" />
+          <cylinder length="0.005" radius="${radius_rotor}"/>  <!-- [m] -->
+          <!--mesh filename="package://morus_description/meshes/propeller_${direction}.dae"
+            scale="0.0025 0.0025 0.0025" /-->
           <!-- <box size="${2*radius_rotor} 0.01 0.005"/> -->
         </geometry>
@@ -169,10 +309,10 @@
     </joint>
     <link name="land_gear_${gear_num}">
-      <!--visual>
+      <visual>
         <origin rpy="0 0 0" xyz="0 0 0"/>
         <geometry>
           <box size="0.01 0.01 0.0001"/>
         </geometry>
-      </visual-->
+      </visual>
       <collision>
         <origin rpy="0 0 0" xyz="0 0 0"/>
